File: eagle/demo/core_mcu.sch (EAGLE design)
At the start: 13 parts, among them IC101 MCU, X302 MALE_2X10-T-VERTICAL_2.54MM

Commit message: kbd module
Parts:
- removed N201: NET_CHANGER-S-0.15MM, be_con_jump:NET_CHANGER-S-0.15MM
- removed N202: NET_CHANGER-S-0.3MM, be_con_jump:NET_CHANGER-S-0.3MM
Connections:
- removed net CORE_CLK: N201.1, X302.2
- removed net CORE_QD: N202.1, X302.4
- net MCU_CLK: now also X302.2; no longer N201.2
- net MCU_QD: now also X302.4; no longer N202.2
Changed lines of the file:
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@@
 <part name="GND1" library="be_supply" deviceset="GND" device=""/>
 <part name="GND2" library="be_supply" deviceset="GND" device=""/>
-<part name="FRAME_NET_CHANGERS1" library="be_frame" deviceset="A4_LANDSCAPE_NET_CHANGERS" device=""/>
 <part name="FRAME_DEVELOPMENT1" library="be_frame" deviceset="A4_LANDSCAPE_DEVELOPMENT" device="">
 <attribute name="DESCRIPTION" value="connectors"/>
@@
 <part name="U$3" library="be_info" deviceset="ARROW_1" device=""/>
 <part name="U$4" library="be_info" deviceset="ARROW_1" device=""/>
-<part name="N201" library="be_con_jump" deviceset="NET_CHANGER" device="-S-0.15MM"/>
-<part name="N202" library="be_con_jump" deviceset="NET_CHANGER" device="-S-0.3MM"/>
-<part name="U$5" library="be_info" deviceset="ARROW_1" device=""/>
-<part name="U$6" library="be_info" deviceset="ARROW_1" device=""/>
-<part name="U$7" library="be_info" deviceset="ARROW_1" device=""/>
-<part name="U$8" library="be_info" deviceset="ARROW_1" device=""/>
 <part name="X301" library="be_con_jump" deviceset="POWER_JACK" device="-T-0">
 <attribute name="FUNCTION" value="PWR IN"/>
@@
 <wire x1="167.64" y1="76.2" x2="172.72" y2="76.2" width="0.1524" layer="91"/>
 <label x="172.72" y="76.2" size="1.27" layer="95" font="fixed" xref="yes"/>
-</segment>
-</net>
-</nets>
-</sheet>
-<sheet>
-<plain>
-</plain>
-<instances>
-<instance part="FRAME_NET_CHANGERS1" gate="G$1" x="0" y="0"/>
-<instance part="N201" gate="G$1" x="170.18" y="58.42" rot="MR0"/>
-<instance part="N202" gate="G$1" x="170.18" y="45.72" rot="MR0"/>
-<instance part="U$5" gate="G$1" x="182.88" y="58.42" rot="MR180"/>
-<instance part="U$6" gate="G$1" x="160.02" y="58.42" rot="MR180"/>
-<instance part="U$7" gate="G$1" x="180.34" y="45.72" rot="R180"/>
-<instance part="U$8" gate="G$1" x="157.48" y="45.72" rot="R180"/>
-</instances>
-<busses>
-</busses>
-<nets>
-<net name="MCU_CLK" class="0">
-<segment>
-<wire x1="162.56" y1="58.42" x2="154.94" y2="58.42" width="0.1524" layer="91"/>
-<label x="154.94" y="58.42" size="1.27" layer="95" font="fixed" rot="MR0" xref="yes"/>
-<pinref part="N201" gate="G$1" pin="2"/>
-</segment>
-</net>
-<net name="CORE_CLK" class="0">
-<segment>
-<pinref part="N201" gate="G$1" pin="1"/>
-<wire x1="177.8" y1="58.42" x2="185.42" y2="58.42" width="0.1524" layer="91"/>
-<label x="185.42" y="58.42" size="1.27" layer="95" font="fixed" rot="MR180" xref="yes"/>
-</segment>
-</net>
-<net name="CORE_QD" class="0">
-<segment>
-<wire x1="177.8" y1="45.72" x2="185.42" y2="45.72" width="0.1524" layer="91"/>
-<label x="185.42" y="45.72" size="1.27" layer="95" font="fixed" xref="yes"/>
-<pinref part="N202" gate="G$1" pin="1"/>
-</segment>
-</net>
-<net name="MCU_QD" class="0">
-<segment>
-<pinref part="N202" gate="G$1" pin="2"/>
-<wire x1="162.56" y1="45.72" x2="154.94" y2="45.72" width="0.1524" layer="91"/>
-<label x="154.94" y="45.72" size="1.27" layer="95" font="fixed" rot="R180" xref="yes"/>
 </segment>
 </net>
@@
 </segment>
 </net>
-<net name="CORE_QD" class="0">
-<segment>
-<wire x1="213.36" y1="68.58" x2="223.52" y2="68.58" width="0.1524" layer="91"/>
-<label x="223.52" y="68.58" size="1.27" layer="95" font="fixed" xref="yes"/>
-<pinref part="X302" gate="G$1" pin="4"/>
-</segment>
-</net>
-<net name="CORE_CLK" class="0">
-<segment>
-<wire x1="213.36" y1="71.12" x2="223.52" y2="71.12" width="0.1524" layer="91"/>
-<label x="223.52" y="71.12" size="1.27" layer="95" font="fixed" xref="yes"/>
-<pinref part="X302" gate="G$1" pin="2"/>
-</segment>
-</net>
 <net name="P5V" class="0">
 <segment>
@@
 </segment>
 </net>
+<net name="MCU_CLK" class="0">
+<segment>
+<wire x1="213.36" y1="71.12" x2="223.52" y2="71.12" width="0.1524" layer="91"/>
+<label x="223.52" y="71.12" size="1.27" layer="95" font="fixed" xref="yes"/>
+<pinref part="X302" gate="G$1" pin="2"/>
+</segment>
+</net>
+<net name="MCU_QD" class="0">
+<segment>
+<wire x1="213.36" y1="68.58" x2="223.52" y2="68.58" width="0.1524" layer="91"/>
+<label x="223.52" y="68.58" size="1.27" layer="95" font="fixed" xref="yes"/>
+<pinref part="X302" gate="G$1" pin="4"/>
+</segment>
+</net>
