File: eagle/demo/core_mcu.sch (EAGLE design)
At the start: 11 parts, among them IC101 MCU, X302 MALE_2X10-T-VERTICAL_2.54MM

Commit message: fix partcodes
Parts:
- C101: PART_CODE_BEL (none) -> C_PAC_S_0805_VAL_100n
- C301: value 10U -> 10u; PART_CODE_BEL (none) -> C_PAC_S_6032_VAL_10u_Vmax_35V
- IC101: value MCU -> SN7495A
- X302: PART_CODE_BEL (none) -> X_PAC_T_MALE_2X10_VERTICAL_PITCH_2mm54
Changed lines of the file:
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@@
 <attribute name="DESCRIPTION" value="core / MCU"/>
 </part>
-<part name="IC101" library="be_logic" deviceset="74*95" device="A" value="MCU"/>
-<part name="C101" library="be_rcl" deviceset="C" device="_S_0805" value="100n"/>
+<part name="IC101" library="be_logic" deviceset="74*95" device="A" value="SN7495A"/>
+<part name="C101" library="be_rcl" deviceset="C" device="_S_0805" value="100n">
+<attribute name="PART_CODE_BEL" value="C_PAC_S_0805_VAL_100n"/>
+</part>
 <part name="GND1" library="be_supply" deviceset="GND" device=""/>
 <part name="GND2" library="be_supply" deviceset="GND" device=""/>
@@
 <part name="H301" library="be_holes" deviceset="HOLE" device="_3.2_PAD"/>
 <part name="H302" library="be_holes" deviceset="HOLE" device="_3.2_PAD"/>
-<part name="C301" library="be_rcl" deviceset="C_POL" device="_S_6032" value="10U"/>
+<part name="C301" library="be_rcl" deviceset="C_POL" device="_S_6032" value="10u">
+<attribute name="PART_CODE_BEL" value="C_PAC_S_6032_VAL_10u_Vmax_35V"/>
+</part>
 <part name="GND6" library="be_supply" deviceset="GND" device=""/>
 <part name="X302" library="be_con_jump" deviceset="MALE_2X10" device="-T-VERTICAL_2.54MM">
 <attribute name="FUNCTION" value="TO SHIELD"/>
+<attribute name="PART_CODE_BEL" value="X_PAC_T_MALE_2X10_VERTICAL_PITCH_2mm54"/>
 </part>
 <part name="U$10" library="be_info" deviceset="ARROW_1" device=""/>

Commit message: fix partcodes
Parts:
- renumbered C301 to C201, FD301 to FD201, FD302 to FD202, H301 to H201, H302 to H202, H303 to H203, H304 to H204, X301 to X201, X302 to X202
Changed lines of the file:
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@@
 <attribute name="DESCRIPTION" value="connectors"/>
 </part>
-<part name="H303" library="be_holes" deviceset="HOLE" device="_3.2_PAD"/>
-<part name="H304" library="be_holes" deviceset="HOLE" device="_3.2_PAD"/>
-<part name="FD301" library="be_marks" deviceset="FIDUCIAL" device="_CROSSHAIR"/>
-<part name="FD302" library="be_marks" deviceset="FIDUCIAL" device="_CROSSHAIR"/>
+<part name="H203" library="be_holes" deviceset="HOLE" device="_3.2_PAD"/>
+<part name="H204" library="be_holes" deviceset="HOLE" device="_3.2_PAD"/>
+<part name="FD201" library="be_marks" deviceset="FIDUCIAL" device="_CROSSHAIR"/>
+<part name="FD202" library="be_marks" deviceset="FIDUCIAL" device="_CROSSHAIR"/>
 <part name="U$3" library="be_info" deviceset="ARROW_1" device=""/>
 <part name="U$4" library="be_info" deviceset="ARROW_1" device=""/>
-<part name="X301" library="be_con_jump" deviceset="POWER_JACK" device="-T-0">
+<part name="X201" library="be_con_jump" deviceset="POWER_JACK" device="-T-0">
 <attribute name="FUNCTION" value="PWR IN"/>
 </part>
 <part name="GND5" library="be_supply" deviceset="GND" device=""/>
-<part name="H301" library="be_holes" deviceset="HOLE" device="_3.2_PAD"/>
-<part name="H302" library="be_holes" deviceset="HOLE" device="_3.2_PAD"/>
-<part name="C301" library="be_rcl" deviceset="C_POL" device="_S_6032" value="10u">
+<part name="H201" library="be_holes" deviceset="HOLE" device="_3.2_PAD"/>
+<part name="H202" library="be_holes" deviceset="HOLE" device="_3.2_PAD"/>
+<part name="C201" library="be_rcl" deviceset="C_POL" device="_S_6032" value="10u">
 <attribute name="PART_CODE_BEL" value="C_PAC_S_6032_VAL_10u_Vmax_35V"/>
 </part>
 <part name="GND6" library="be_supply" deviceset="GND" device=""/>
-<part name="X302" library="be_con_jump" deviceset="MALE_2X10" device="-T-VERTICAL_2.54MM">
+<part name="X202" library="be_con_jump" deviceset="MALE_2X10" device="-T-VERTICAL_2.54MM">
 <attribute name="FUNCTION" value="TO SHIELD"/>
 <attribute name="PART_CODE_BEL" value="X_PAC_T_MALE_2X10_VERTICAL_PITCH_2mm54"/>
@@
 <attribute name="STATUS" x="132.08" y="19" size="1.778" layer="100" font="fixed"/>
 </instance>
-<instance part="H303" gate="G$1" x="50.8" y="30.48" smashed="yes">
+<instance part="H203" gate="G$1" x="50.8" y="30.48" smashed="yes">
 <attribute name="NAME" x="53.975" y="31.75" size="1.778" layer="95" font="fixed"/>
 <attribute name="VALUE" x="53.975" y="29.21" size="1.778" layer="96" font="fixed"/>
 </instance>
-<instance part="H304" gate="G$1" x="50.8" y="17.78" smashed="yes">
+<instance part="H204" gate="G$1" x="50.8" y="17.78" smashed="yes">
 <attribute name="NAME" x="53.975" y="19.05" size="1.778" layer="95" font="fixed"/>
 <attribute name="VALUE" x="53.975" y="16.51" size="1.778" layer="96" font="fixed"/>
 </instance>
-<instance part="FD301" gate="FD" x="83.82" y="30.48" smashed="yes">
+<instance part="FD201" gate="FD" x="83.82" y="30.48" smashed="yes">
 <attribute name="NAME" x="78.74" y="33.655" size="1.27" layer="95" font="fixed"/>
 </instance>
-<instance part="FD302" gate="FD" x="83.82" y="17.78" smashed="yes">
+<instance part="FD202" gate="FD" x="83.82" y="17.78" smashed="yes">
 <attribute name="NAME" x="78.74" y="20.955" size="1.27" layer="95" font="fixed"/>
 </instance>
-<instance part="X301" gate="G$1" x="144.78" y="60.96" smashed="yes">
+<instance part="X201" gate="G$1" x="144.78" y="60.96" smashed="yes">
 <attribute name="FUNCTION" x="137.16" y="71.12" size="2.54" layer="96" font="fixed"/>
 <attribute name="NAME" x="137.16" y="67.945" size="1.27" layer="95" font="fixed"/>
@@
 <attribute name="VALUE" x="150.622" y="46.355" size="1.27" layer="96" font="fixed"/>
 </instance>
-<instance part="H301" gate="G$1" x="22.86" y="30.48" smashed="yes">
+<instance part="H201" gate="G$1" x="22.86" y="30.48" smashed="yes">
 <attribute name="NAME" x="26.035" y="31.75" size="1.778" layer="95" font="fixed"/>
 <attribute name="VALUE" x="26.035" y="29.21" size="1.778" layer="96" font="fixed"/>
 </instance>
-<instance part="H302" gate="G$1" x="22.86" y="17.78" smashed="yes">
+<instance part="H202" gate="G$1" x="22.86" y="17.78" smashed="yes">
 <attribute name="NAME" x="26.035" y="19.05" size="1.778" layer="95" font="fixed"/>
 <attribute name="VALUE" x="26.035" y="16.51" size="1.778" layer="96" font="fixed"/>
 </instance>
-<instance part="C301" gate="G$1" x="162.56" y="58.42"/>
+<instance part="C201" gate="G$1" x="162.56" y="58.42"/>
 <instance part="GND6" gate="1" x="162.56" y="48.26" smashed="yes">
 <attribute name="VALUE" x="160.782" y="46.355" size="1.27" layer="96" font="fixed"/>
 </instance>
-<instance part="X302" gate="G$1" x="208.28" y="60.96">
+<instance part="X202" gate="G$1" x="208.28" y="60.96">
 <attribute name="FUNCTION" x="200.66" y="81.28" size="2.54" layer="96" font="fixed"/>
 </instance>
@@
 <net name="GND" class="0">
 <segment>
-<pinref part="X301" gate="G$1" pin="1"/>
+<pinref part="X201" gate="G$1" pin="1"/>
 <wire x1="149.86" y1="58.42" x2="152.4" y2="58.42" width="0.1524" layer="91"/>
 <wire x1="152.4" y1="58.42" x2="152.4" y2="50.8" width="0.1524" layer="91"/>
@@
 </segment>
 <segment>
-<pinref part="C301" gate="G$1" pin="-"/>
+<pinref part="C201" gate="G$1" pin="-"/>
 <wire x1="162.56" y1="53.34" x2="162.56" y2="50.8" width="0.1524" layer="91"/>
 <pinref part="GND6" gate="1" pin="GND"/>
 </segment>
 <segment>
-<pinref part="X302" gate="G$1" pin="1"/>
+<pinref part="X202" gate="G$1" pin="1"/>
 <wire x1="203.2" y1="71.12" x2="195.58" y2="71.12" width="0.1524" layer="91"/>
 <wire x1="195.58" y1="71.12" x2="195.58" y2="68.58" width="0.1524" layer="91"/>
-<pinref part="X302" gate="G$1" pin="3"/>
+<pinref part="X202" gate="G$1" pin="3"/>
 <wire x1="195.58" y1="68.58" x2="203.2" y2="68.58" width="0.1524" layer="91"/>
 <pinref part="GND7" gate="1" pin="GND"/>
@@
 <net name="P5V" class="0">
 <segment>
-<pinref part="X301" gate="G$1" pin="3"/>
+<pinref part="X201" gate="G$1" pin="3"/>
 <label x="166.37" y="64.135" size="1.27" layer="95" font="fixed"/>
 <wire x1="149.86" y1="63.5" x2="162.56" y2="63.5" width="0.1524" layer="91"/>
-<pinref part="C301" gate="G$1" pin="+"/>
+<pinref part="C201" gate="G$1" pin="+"/>
 <wire x1="162.56" y1="63.5" x2="170.18" y2="63.5" width="0.1524" layer="91"/>
 <wire x1="162.56" y1="63.5" x2="162.56" y2="60.96" width="0.1524" layer="91"/>
@@
 <wire x1="213.36" y1="71.12" x2="223.52" y2="71.12" width="0.1524" layer="91"/>
 <label x="223.52" y="71.12" size="1.27" layer="95" font="fixed" xref="yes"/>
-<pinref part="X302" gate="G$1" pin="2"/>
+<pinref part="X202" gate="G$1" pin="2"/>
 </segment>
 </net>
@@
 <wire x1="213.36" y1="68.58" x2="223.52" y2="68.58" width="0.1524" layer="91"/>
 <label x="223.52" y="68.58" size="1.27" layer="95" font="fixed" xref="yes"/>
-<pinref part="X302" gate="G$1" pin="4"/>
+<pinref part="X202" gate="G$1" pin="4"/>
 </segment>
 </net>
