File: eagle/demo/product.brd (EAGLE design)
At the start: 80 x 50 mm, 11 parts, among them IC101 MCU, T201 BC548C, X201 CLAMP_1X2-T-2.5MM

Commit message: step 6: route pwr
Routing:
- net GND: track 0.00 -> 6.33 mm, vias 0 -> 4
- net P5V: track 0.00 -> 4.94 mm, vias 0 -> 3
- added copper zone on layer 15, net GND
- added copper zone on layer 2, net P5V

Commit message: step 7: finish routing
Routing:
- net KBD_OUT: track 0.00 -> 55.7 mm
- net LED_DRV_IN: track 0.00 -> 27.7 mm
- net KBD_RC: track 0.00 -> 13.4 mm
- net LED_DRV_OUT: track 0.00 -> 11.7 mm
- net LED_DRV_B: track 0.00 -> 4.85 mm
- net LED_DRV_C: track 0.00 -> 4.54 mm
Other:
- outline, holes or cut-outs redrawn
- board text added: "LIGHT SAVER"
Changed lines of the file:
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@@
 <wire x1="60" y1="50" x2="0" y2="50" width="0" layer="20"/>
 <wire x1="0" y1="50" x2="0" y2="0" width="0" layer="20"/>
-<circle x="30" y="30" radius="10" width="0.15" layer="54"/>
+<circle x="30" y="30" radius="10" width="0.15" layer="20"/>
+<text x="21.4" y="45.2" size="1.5" layer="21" font="vector" ratio="13">LIGHT SAVER</text>
 </plain>
 <attributes>
@@
 <param name="AutoGrid" value="1"/>
 <param name="Efforts" value="0"/>
-<param name="TopRouterVariant" value="1"/>
+<param name="TopRouterVariant" value="0"/>
 <param name="tpViaShape" value="round"/>
-<param name="PrefDir.1" value="a"/>
-<param name="PrefDir.2" value="0"/>
+<param name="PrefDir.1" value="-"/>
+<param name="PrefDir.2" value="a"/>
 <param name="PrefDir.3" value="0"/>
 <param name="PrefDir.4" value="0"/>
@@
 <param name="PrefDir.13" value="0"/>
 <param name="PrefDir.14" value="0"/>
-<param name="PrefDir.15" value="0"/>
-<param name="PrefDir.16" value="a"/>
+<param name="PrefDir.15" value="a"/>
+<param name="PrefDir.16" value="|"/>
 <param name="cfVia" value="8"/>
 <param name="cfNonPref" value="5"/>
@@
 <contactref element="S301" pad="A"/>
 <contactref element="S301" pad="A1"/>
-<wire x1="11.35" y1="40.48" x2="43.87" y2="23.22" width="0" layer="19" extent="1-1"/>
-<wire x1="4.55" y1="40.48" x2="11.35" y2="40.48" width="0" layer="19" extent="1-1"/>
+<wire x1="41" y1="26" x2="43.5" y2="23.5" width="0.15" layer="1"/>
+<wire x1="41" y1="41" x2="41" y2="26" width="0.15" layer="1"/>
+<wire x1="12" y1="41" x2="41" y2="41" width="0.15" layer="1"/>
+<wire x1="11.5" y1="40.5" x2="12" y2="41" width="0.15" layer="1"/>
+<wire x1="43.5" y1="23.5" x2="43.87" y2="23.22" width="0.15" layer="1"/>
+<wire x1="11.5" y1="40.5" x2="11.35" y2="40.48" width="0.15" layer="1"/>
+<wire x1="11" y1="40.5" x2="5" y2="40.5" width="0.15" layer="1"/>
+<wire x1="5" y1="40.5" x2="4.55" y2="40.48" width="0.15" layer="1"/>
+<wire x1="11" y1="40.5" x2="11.35" y2="40.48" width="0.15" layer="1"/>
 </signal>
 <signal name="LED_DRV_IN">
 <contactref element="IC101" pad="10"/>
 <contactref element="R201" pad="1"/>
-<wire x1="20.95" y1="9" x2="43.87" y2="20.68" width="0" layer="19" extent="1-1"/>
+<wire x1="31" y1="19" x2="21" y2="9" width="0.15" layer="1"/>
+<wire x1="42" y1="19" x2="31" y2="19" width="0.15" layer="1"/>
+<wire x1="43.5" y1="20.5" x2="42" y2="19" width="0.15" layer="1"/>
+<wire x1="21" y1="9" x2="20.95" y2="9" width="0.15" layer="1"/>
+<wire x1="43.5" y1="20.5" x2="43.87" y2="20.68" width="0.15" layer="1"/>
 </signal>
 <signal name="LED_DRV_B">
 <contactref element="R201" pad="2"/>
 <contactref element="T201" pad="1"/>
-<wire x1="19.05" y1="9" x2="20.05" y2="12.9" width="0" layer="19" extent="1-1"/>
+<wire x1="20" y1="9" x2="20" y2="12.5" width="0.15" layer="1"/>
+<wire x1="19.05" y1="9" x2="20" y2="9" width="0.15" layer="1"/>
+<wire x1="20" y1="12.5" x2="20.05" y2="12.9" width="0.15" layer="1"/>
 </signal>
 <signal name="LED_DRV_C">
 <contactref element="T201" pad="3"/>
 <contactref element="R202" pad="1"/>
-<wire x1="16.91" y1="15.43" x2="21" y2="15.1" width="0" layer="19" extent="1-1"/>
+<wire x1="17" y1="15" x2="21" y2="15" width="0.15" layer="1"/>
+<wire x1="21" y1="15" x2="21" y2="15.1" width="0.15" layer="1"/>
+<wire x1="17" y1="15" x2="16.91" y2="15.43" width="0.15" layer="1"/>
 </signal>
 <signal name="LED_DRV_OUT">
 <contactref element="R202" pad="2"/>
 <contactref element="X201" pad="2"/>
-<wire x1="7.98" y1="19.75" x2="16.91" y2="13.53" width="0" layer="19" extent="1-1"/>
+<wire x1="11" y1="19.5" x2="16.5" y2="14" width="0.15" layer="1"/>
+<wire x1="8" y1="19.5" x2="11" y2="19.5" width="0.15" layer="1"/>
+<wire x1="16.5" y1="14" x2="16.91" y2="13.53" width="0.15" layer="1"/>
+<wire x1="8" y1="19.5" x2="7.98" y2="19.75" width="0.15" layer="1"/>
 </signal>
 <signal name="KBD_RC">
@@
 <contactref element="S301" pad="B"/>
 <contactref element="S301" pad="B1"/>
-<wire x1="9.95" y1="33" x2="11.35" y2="36.48" width="0" layer="19" extent="1-1"/>
-<wire x1="13.05" y1="33" x2="9.95" y2="33" width="0" layer="19" extent="1-1"/>
-<wire x1="4.55" y1="36.48" x2="9.95" y2="33" width="0" layer="19" extent="1-1"/>
+<wire x1="13.05" y1="33" x2="11.5" y2="33" width="0.15" layer="1"/>
+<wire x1="11.5" y1="33" x2="9.95" y2="33" width="0.15" layer="1"/>
+<wire x1="11.5" y1="36" x2="11.5" y2="33" width="0.15" layer="1"/>
+<wire x1="11.5" y1="36" x2="11.35" y2="36.48" width="0.15" layer="1"/>
+<wire x1="11" y1="36.5" x2="5" y2="36.5" width="0.15" layer="1"/>
+<wire x1="5" y1="36.5" x2="4.55" y2="36.48" width="0.15" layer="1"/>
+<wire x1="11" y1="36.5" x2="11.35" y2="36.48" width="0.15" layer="1"/>
 </signal>
 </signals>

Commit message: step 8: replace MCU package
Parts:
- IC101: device be_logic:T_NDIP14 -> be_logic:S_SO14
- moved C101 5.02 mm to (47.4, 11.9)
Routing:
- net KBD_OUT: track 55.7 -> 59.8 mm
- net GND: track 6.33 -> 8.00 mm, vias 4 -> 5
- net P5V: track 4.94 -> 6.57 mm, vias 3 -> 4
Changed lines of the file:
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@@
 <attribute name="PART_CODE_EXT" value="" x="9" y="15" size="1.778" layer="27" rot="R180" display="off"/>
 </element>
-<element name="C101" library="be_rcl" package="S_0805" value="100n" x="47.76" y="6.91">
-<attribute name="UPDATED" value="" x="47.76" y="6.91" size="1.778" layer="27" display="off"/>
-<attribute name="PART_CODE_BEL" value="C_PAC_S_0805_VAL_" x="47.76" y="6.91" size="1.778" layer="27" display="off"/>
-<attribute name="BOM" value="YES" x="47.76" y="6.91" size="1.778" layer="27" display="off"/>
-<attribute name="FUNCTION" value="" x="47.76" y="6.91" size="1.778" layer="27" display="off"/>
-<attribute name="COMMISSIONED" value="2013-08-30" x="47.76" y="6.91" size="1.778" layer="27" display="off"/>
-<attribute name="PART_CODE_EXT" value="" x="47.76" y="6.91" size="1.778" layer="27" display="off"/>
+<element name="C101" library="be_rcl" package="S_0805" value="100n" x="47.36" y="11.91">
+<attribute name="UPDATED" value="" x="47.36" y="11.91" size="1.778" layer="27" display="off"/>
+<attribute name="PART_CODE_BEL" value="C_PAC_S_0805_VAL_" x="47.36" y="11.91" size="1.778" layer="27" display="off"/>
+<attribute name="BOM" value="YES" x="47.36" y="11.91" size="1.778" layer="27" display="off"/>
+<attribute name="FUNCTION" value="" x="47.36" y="11.91" size="1.778" layer="27" display="off"/>
+<attribute name="COMMISSIONED" value="2013-08-30" x="47.36" y="11.91" size="1.778" layer="27" display="off"/>
+<attribute name="PART_CODE_EXT" value="" x="47.36" y="11.91" size="1.778" layer="27" display="off"/>
 </element>
 <element name="C301" library="be_rcl" package="S_0805" value="100n" x="14" y="33">
@@
 <attribute name="PART_CODE_EXT" value="" x="14" y="33" size="1.778" layer="27" display="off"/>
 </element>
-<element name="IC101" library="be_logic" package="T_NDIP14" value="MCU" x="47.68" y="18.14" rot="R90">
+<element name="IC101" library="be_logic" package="S_SO14" value="MCU" x="47.68" y="18.14" rot="R90">
 <attribute name="UPDATED" value="" x="47.68" y="18.14" size="1.778" layer="27" rot="R90" display="off"/>
-<attribute name="PART_CODE_BEL" value="IC_PAC_T_NDIP14_VAL_SN7495A" x="47.68" y="18.14" size="1.778" layer="27" rot="R90" display="off"/>
-<attribute name="BOM" value="YES" x="47.68" y="18.14" size="1.778" layer="27" rot="R90" display="off"/>
+<attribute name="PART_CODE_BEL" value="" x="47.68" y="18.14" size="1.778" layer="27" rot="R90" display="off"/>
+<attribute name="BOM" value="" x="47.68" y="18.14" size="1.778" layer="27" rot="R90" display="off"/>
 <attribute name="FUNCTION" value="" x="47.68" y="18.14" size="1.778" layer="27" rot="R90" display="off"/>
-<attribute name="COMMISSIONED" value="2015-05-19" x="47.68" y="18.14" size="1.778" layer="27" rot="R90" display="off"/>
+<attribute name="COMMISSIONED" value="" x="47.68" y="18.14" size="1.778" layer="27" rot="R90" display="off"/>
 <attribute name="PART_CODE_EXT" value="" x="47.68" y="18.14" size="1.778" layer="27" rot="R90" display="off"/>
 </element>
@@
 <vertex x="0" y="0"/>
 </polygon>
-<wire x1="46.81" y1="6.91" x2="46.72" y2="7" width="0.15" layer="1"/>
-<wire x1="46.72" y1="7" x2="45.6" y2="7" width="0.15" layer="1"/>
-<via x="45.6" y="7" extent="1-16" drill="0.3"/>
+<wire x1="46.41" y1="11.91" x2="46.32" y2="12" width="0.15" layer="1"/>
+<wire x1="46.32" y1="12" x2="45.2" y2="12" width="0.15" layer="1"/>
+<via x="45.2" y="12" extent="1-16" drill="0.3"/>
 <wire x1="8.05" y1="33" x2="6.6" y2="33" width="0.15" layer="1"/>
 <via x="6.6" y="33" extent="1-16" drill="0.3"/>
@@
 <wire x1="11.4" y1="14.9" x2="11.4" y2="12.8" width="0.15" layer="1"/>
 <via x="11.4" y="12.8" extent="1-16" drill="0.3"/>
+<wire x1="44.6066" y1="14.33" x2="44.5366" y2="14.4" width="0.15" layer="1"/>
+<wire x1="44.5366" y1="14.4" x2="43" y2="14.4" width="0.15" layer="1"/>
+<via x="43" y="14.4" extent="1-16" drill="0.3"/>
 </signal>
 <signal name="GND">
@@
 <vertex x="0" y="0"/>
 </polygon>
-<wire x1="48.71" y1="6.91" x2="48.8" y2="7" width="0.15" layer="1"/>
-<wire x1="48.8" y1="7" x2="50" y2="7" width="0.15" layer="1"/>
-<via x="50" y="7" extent="1-16" drill="0.3"/>
+<wire x1="48.31" y1="11.91" x2="48.4" y2="12" width="0.15" layer="1"/>
+<wire x1="48.4" y1="12" x2="49.6" y2="12" width="0.15" layer="1"/>
+<via x="49.6" y="12" extent="1-16" drill="0.3"/>
 <wire x1="6.5" y1="15" x2="6.3" y2="15.2" width="0.15" layer="1"/>
 <wire x1="6.3" y1="15.2" x2="4.4" y2="15.2" width="0.15" layer="1"/>
@@
 <wire x1="14.95" y1="33" x2="16.4" y2="33" width="0.15" layer="1"/>
 <via x="16.4" y="33" extent="1-16" drill="0.3"/>
+<wire x1="50.7534" y1="21.95" x2="50.8034" y2="22" width="0.15" layer="1"/>
+<wire x1="50.8034" y1="22" x2="52.4" y2="22" width="0.15" layer="1"/>
+<via x="52.4" y="22" extent="1-16" drill="0.3"/>
 </signal>
 <signal name="KBD_OUT">
@@
 <contactref element="S301" pad="A"/>
 <contactref element="S301" pad="A1"/>
-<wire x1="41" y1="26" x2="43.5" y2="23.5" width="0.15" layer="1"/>
-<wire x1="41" y1="41" x2="41" y2="26" width="0.15" layer="1"/>
+<wire x1="41" y1="41" x2="41" y2="22" width="0.15" layer="1"/>
 <wire x1="12" y1="41" x2="41" y2="41" width="0.15" layer="1"/>
 <wire x1="11.5" y1="40.5" x2="12" y2="41" width="0.15" layer="1"/>
-<wire x1="43.5" y1="23.5" x2="43.87" y2="23.22" width="0.15" layer="1"/>
 <wire x1="11.5" y1="40.5" x2="11.35" y2="40.48" width="0.15" layer="1"/>
 <wire x1="11" y1="40.5" x2="5" y2="40.5" width="0.15" layer="1"/>
 <wire x1="5" y1="40.5" x2="4.55" y2="40.48" width="0.15" layer="1"/>
 <wire x1="11" y1="40.5" x2="11.35" y2="40.48" width="0.15" layer="1"/>
+<wire x1="41" y1="22" x2="42.32" y2="20.68" width="0.15" layer="1"/>
+<wire x1="42.32" y1="20.68" x2="44.6066" y2="20.68" width="0.15" layer="1"/>
 </signal>
 <signal name="LED_DRV_IN">
@@
 <wire x1="31" y1="19" x2="21" y2="9" width="0.15" layer="1"/>
 <wire x1="42" y1="19" x2="31" y2="19" width="0.15" layer="1"/>
-<wire x1="43.5" y1="20.5" x2="42" y2="19" width="0.15" layer="1"/>
 <wire x1="21" y1="9" x2="20.95" y2="9" width="0.15" layer="1"/>
-<wire x1="43.5" y1="20.5" x2="43.87" y2="20.68" width="0.15" layer="1"/>
+<wire x1="42" y1="19" x2="42.41" y2="19.41" width="0.15" layer="1"/>
+<wire x1="42.41" y1="19.41" x2="44.6066" y2="19.41" width="0.15" layer="1"/>
 </signal>
 <signal name="LED_DRV_B">
