File: eagle/demo/core_mcu.brd (EAGLE design)
At the start: 70 x 50 mm, 14 parts, among them IC101 MCU, X302 MALE_2X10-T-VERTICAL_2.54MM

Commit message: kbd module
Parts:
- removed N201: NET_CHANGER-S-0.15MM, be_con_jump:S_NET_CHANGER_0.15MM
- removed N202: NET_CHANGER-S-0.3MM, be_con_jump:S_NET_CHANGER_0.3MM
Connections:
- removed net CORE_CLK: N201.1, X302.2
- removed net CORE_QD: N202.1, X302.4
- net MCU_CLK: now also X302.2; no longer N201.2
- net MCU_QD: now also X302.4; no longer N202.2
Routing:
- net CORE_CLK: track 17.0 -> 0.00 mm
- net CORE_QD: track 16.5 -> 0.00 mm
- net MCU_CLK: track 26.6 -> 21.7 mm
- net MCU_QD: track 17.8 -> 13.5 mm
Changed lines of the file:
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@@
 <attribute name="VALUE" x="34.365" y="29.731" size="1" layer="27" font="vector" ratio="13" rot="R270"/>
-</element>
-<element name="N201" library="be_con_jump" package="S_NET_CHANGER_0.15MM" value="NET_CHANGER-S-0.15MM" x="52" y="29" smashed="yes" rot="R180">
-<attribute name="FUNCTION" value="" x="52" y="29" size="1.778" layer="27" rot="R180" display="off"/>
-<attribute name="PART_CODE_EXT" value="" x="52" y="29" size="1.778" layer="27" rot="R180" display="off"/>
-<attribute name="COMMISSIONED" value="2013-08-30" x="52" y="29" size="1.778" layer="27" rot="R180" display="off"/>
-<attribute name="BOM" value="NO" x="52" y="29" size="1.778" layer="27" rot="R180" display="off"/>
-<attribute name="PART_CODE_BEL" value="N_PAC_S_NET_CHANGER_0.15MM" x="52" y="29" size="1.778" layer="27" rot="R180" display="off"/>
-<attribute name="UPDATED" value="" x="52" y="29" size="1.778" layer="27" rot="R180" display="off"/>
-<attribute name="NAME" x="53" y="29.8" size="0.5" layer="25" font="vector" ratio="13" rot="R180"/>
-</element>
-<element name="N202" library="be_con_jump" package="S_NET_CHANGER_0.3MM" value="NET_CHANGER-S-0.3MM" x="52" y="27" smashed="yes" rot="R180">
-<attribute name="FUNCTION" value="" x="52" y="27" size="1.778" layer="27" rot="R180" display="off"/>
-<attribute name="PART_CODE_EXT" value="" x="52" y="27" size="1.778" layer="27" rot="R180" display="off"/>
-<attribute name="COMMISSIONED" value="2014-04-09" x="52" y="27" size="1.778" layer="27" rot="R180" display="off"/>
-<attribute name="BOM" value="NO" x="52" y="27" size="1.778" layer="27" rot="R180" display="off"/>
-<attribute name="PART_CODE_BEL" value="N_PAC_S_NET_CHANGER_0.3MM" x="52" y="27" size="1.778" layer="27" rot="R180" display="off"/>
-<attribute name="UPDATED" value="" x="52" y="27" size="1.778" layer="27" rot="R180" display="off"/>
-<attribute name="NAME" x="53.1" y="26.7" size="0.5" layer="25" font="vector" ratio="13" rot="R180"/>
 </element>
 <element name="X301" library="be_con_jump" package="T_POWER_JACK_SPC4077" value="" x="9.98" y="35.35" smashed="yes">
@@
 <signal name="MCU_CLK">
 <contactref element="IC101" pad="9"/>
-<contactref element="N201" pad="2"/>
 <wire x1="38.81" y1="17.92" x2="36.88" y2="17.92" width="0.15" layer="1"/>
 <wire x1="36.88" y1="17.92" x2="36.4" y2="18.4" width="0.15" layer="1"/>
@@
 <wire x1="44.8" y1="22" x2="44.8" y2="27" width="0.15" layer="1"/>
 <wire x1="44.8" y1="27" x2="46.8" y2="29" width="0.15" layer="1"/>
-<wire x1="46.8" y1="29" x2="51.7" y2="29" width="0.15" layer="1"/>
+<contactref element="X302" pad="2"/>
+<wire x1="46.8" y1="29" x2="64.27" y2="36.43" width="0" layer="19" extent="1-1"/>
 </signal>
 <signal name="MCU_QD">
 <contactref element="IC101" pad="10"/>
-<contactref element="N202" pad="2"/>
 <wire x1="38.81" y1="20.46" x2="44.66" y2="20.46" width="0.3" layer="1"/>
 <wire x1="44.66" y1="20.46" x2="45.6" y2="21.4" width="0.3" layer="1"/>
 <wire x1="45.6" y1="21.4" x2="45.6" y2="25.2" width="0.3" layer="1"/>
 <wire x1="45.6" y1="25.2" x2="47.4" y2="27" width="0.3" layer="1"/>
-<wire x1="47.4" y1="27" x2="51.7" y2="27" width="0.3" layer="1"/>
-</signal>
-<signal name="CORE_CLK">
-<contactref element="N201" pad="1"/>
-<contactref element="X302" pad="2"/>
-<wire x1="52.3" y1="29" x2="55" y2="29" width="0.15" layer="1"/>
-<wire x1="55" y1="29" x2="56" y2="30" width="0.15" layer="1"/>
-<wire x1="56" y1="30" x2="56" y2="33.4" width="0.15" layer="1"/>
-<wire x1="56" y1="33.4" x2="57.8" y2="35.2" width="0.15" layer="1"/>
-<wire x1="57.8" y1="35.2" x2="63.04" y2="35.2" width="0.15" layer="1"/>
-<wire x1="63.04" y1="35.2" x2="64.27" y2="36.43" width="0.15" layer="1"/>
-</signal>
-<signal name="CORE_QD">
-<contactref element="N202" pad="1"/>
 <contactref element="X302" pad="4"/>
-<wire x1="52.3" y1="27" x2="55" y2="27" width="0.3" layer="1"/>
-<wire x1="55" y1="27" x2="56.6" y2="28.6" width="0.3" layer="1"/>
-<wire x1="56.6" y1="28.6" x2="56.6" y2="31.4" width="0.3" layer="1"/>
-<wire x1="56.6" y1="31.4" x2="57.6" y2="32.4" width="0.3" layer="1"/>
-<wire x1="57.6" y1="32.4" x2="62.78" y2="32.4" width="0.3" layer="1"/>
-<wire x1="62.78" y1="32.4" x2="64.27" y2="33.89" width="0.3" layer="1"/>
+<wire x1="47.4" y1="27" x2="64.27" y2="33.89" width="0" layer="19" extent="1-1"/>
 </signal>
 </signals>

Commit message: finished core
Routing:
- net MCU_CLK: track 21.7 -> 42.4 mm
- net MCU_QD: track 13.5 -> 33.3 mm
- added copper zone on layer 2, net P5V
Changed lines of the file:
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@@
 <layers>
 <layer number="1" name="Top" color="4" fill="1" visible="yes" active="yes"/>
-<layer number="2" name="Route2" color="1" fill="3" visible="no" active="yes"/>
+<layer number="2" name="Route2" color="1" fill="3" visible="yes" active="yes"/>
 <layer number="3" name="Route3" color="4" fill="3" visible="no" active="no"/>
 <layer number="4" name="Route4" color="1" fill="4" visible="no" active="no"/>
@@
 <wire x1="17.4" y1="36.3" x2="16.45" y2="35.35" width="1" layer="1"/>
 <wire x1="16.45" y1="35.35" x2="12.98" y2="35.35" width="1" layer="1"/>
-<wire x1="39.2" y1="33.4" x2="38.81" y2="30.62" width="0" layer="19" extent="1-1"/>
-<wire x1="17.4" y1="36.3" x2="37.95" y2="34" width="0" layer="19" extent="1-1"/>
+<polygon width="0.15" layer="2">
+<vertex x="12" y="40"/>
+<vertex x="42" y="40"/>
+<vertex x="42" y="28"/>
+<vertex x="12" y="28"/>
+</polygon>
 </signal>
 <signal name="GND">
@@
 <wire x1="44.4" y1="21.6" x2="44.8" y2="22" width="0.15" layer="1"/>
 <wire x1="44.8" y1="22" x2="44.8" y2="27" width="0.15" layer="1"/>
-<wire x1="44.8" y1="27" x2="46.8" y2="29" width="0.15" layer="1"/>
 <contactref element="X302" pad="2"/>
-<wire x1="46.8" y1="29" x2="64.27" y2="36.43" width="0" layer="19" extent="1-1"/>
+<wire x1="44.8" y1="27" x2="53" y2="35.2" width="0.15" layer="1"/>
+<wire x1="53" y1="35.2" x2="63.2" y2="35.2" width="0.15" layer="1"/>
+<wire x1="63.2" y1="35.2" x2="64.27" y2="36.27" width="0.15" layer="1"/>
+<wire x1="64.27" y1="36.27" x2="64.27" y2="36.43" width="0.15" layer="1"/>
 </signal>
 <signal name="MCU_QD">
@@
 <wire x1="44.66" y1="20.46" x2="45.6" y2="21.4" width="0.3" layer="1"/>
 <wire x1="45.6" y1="21.4" x2="45.6" y2="25.2" width="0.3" layer="1"/>
-<wire x1="45.6" y1="25.2" x2="47.4" y2="27" width="0.3" layer="1"/>
 <contactref element="X302" pad="4"/>
-<wire x1="47.4" y1="27" x2="64.27" y2="33.89" width="0" layer="19" extent="1-1"/>
+<wire x1="45.6" y1="25.2" x2="53" y2="32.6" width="0.3" layer="1"/>
+<wire x1="53" y1="32.6" x2="63" y2="32.6" width="0.3" layer="1"/>
+<wire x1="63" y1="32.6" x2="64.27" y2="33.87" width="0.3" layer="1"/>
+<wire x1="64.27" y1="33.87" x2="64.27" y2="33.89" width="0.3" layer="1"/>
 </signal>
 </signals>

Commit message: fix partcodes
Parts:
- C301: value 10U -> 10u
- IC101: value MCU -> SN7495A
Changed lines of the file:
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@@
 <attribute name="COMMISSIONED" value="2013-08-30" x="37" y="34" size="1.778" layer="27" rot="R180" display="off"/>
 <attribute name="BOM" value="YES" x="37" y="34" size="1.778" layer="27" rot="R180" display="off"/>
-<attribute name="PART_CODE_BEL" value="C_PAC_S_0805_VAL_" x="37" y="34" size="1.778" layer="27" rot="R180" display="off"/>
+<attribute name="PART_CODE_BEL" value="C_PAC_S_0805_VAL_100n" x="37" y="34" size="1.778" layer="27" rot="R180" display="off"/>
 <attribute name="UPDATED" value="" x="37" y="34" size="1.778" layer="27" rot="R180" display="off"/>
 <attribute name="NAME" x="39" y="36.5" size="1" layer="25" font="vector" ratio="13" rot="R180"/>
@@
 <attribute name="UPDATED" value="" x="5" y="45" size="1.778" layer="27" display="off"/>
 </element>
-<element name="IC101" library="be_logic" package="T_NDIP14" value="MCU" x="35" y="23" smashed="yes" rot="R270">
+<element name="IC101" library="be_logic" package="T_NDIP14" value="SN7495A" x="35" y="23" smashed="yes" rot="R270">
 <attribute name="FUNCTION" value="" x="35" y="23" size="1.778" layer="27" rot="R270" display="off"/>
 <attribute name="PART_CODE_EXT" value="" x="35" y="23" size="1.778" layer="27" rot="R270" display="off"/>
@@
 <attribute name="UPDATED" value="" x="65" y="5" size="1" layer="27" font="vector" ratio="13" display="off"/>
 </element>
-<element name="C301" library="be_rcl" package="S_6032" value="10U" x="17.4" y="33.8" rot="R270">
+<element name="C301" library="be_rcl" package="S_6032" value="10u" x="17.4" y="33.8" rot="R270">
 <attribute name="FUNCTION" value="" x="17.4" y="33.8" size="1" layer="27" font="vector" ratio="15" rot="R270" display="off"/>
 <attribute name="PART_CODE_EXT" value="" x="17.4" y="33.8" size="1" layer="27" font="vector" ratio="15" rot="R270" display="off"/>
 <attribute name="COMMISSIONED" value="2013-08-30" x="17.4" y="33.8" size="1" layer="27" font="vector" ratio="15" rot="R270" display="off"/>
 <attribute name="BOM" value="YES" x="17.4" y="33.8" size="1" layer="27" font="vector" ratio="15" rot="R270" display="off"/>
-<attribute name="PART_CODE_BEL" value="C_PAC_S_6032_VAL_" x="17.4" y="33.8" size="1" layer="27" font="vector" ratio="15" rot="R270" display="off"/>
+<attribute name="PART_CODE_BEL" value="C_PAC_S_6032_VAL_10u_Vmax_35V" x="17.4" y="33.8" size="1" layer="27" font="vector" ratio="15" rot="R270" display="off"/>
 <attribute name="UPDATED" value="" x="17.4" y="33.8" size="1" layer="27" font="vector" ratio="15" rot="R270" display="off"/>
 </element>
@@
 <attribute name="COMMISSIONED" value="2013-08-30" x="63" y="25" size="1.5" layer="27" font="vector" ratio="15" rot="R270" display="off"/>
 <attribute name="BOM" value="YES" x="63" y="25" size="1.5" layer="27" font="vector" ratio="15" rot="R270" display="off"/>
-<attribute name="PART_CODE_BEL" value="X_PAC_T_MALE_2X10_VERTICAL_GRID_2.54mm" x="63" y="25" size="1.5" layer="27" font="vector" ratio="15" rot="R270" display="off"/>
+<attribute name="PART_CODE_BEL" value="X_PAC_T_MALE_2X10_VERTICAL_PITCH_2mm54" x="63" y="25" size="1.5" layer="27" font="vector" ratio="15" rot="R270" display="off"/>
 <attribute name="UPDATED" value="" x="63" y="25" size="1.5" layer="27" font="vector" ratio="15" rot="R270" display="off"/>
 <attribute name="NAME" x="60.4" y="38.6" size="1" layer="25" font="vector" ratio="13"/>

Commit message: fix partcodes
Parts:
- renumbered C301 to C201, FD301 to FD201, FD302 to FD202, H301 to H201, H302 to H202, H303 to H203, H304 to H204, X301 to X201, X302 to X202
Changed lines of the file:
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@@
 <attribute name="VALUE" x="39" y="38" size="1" layer="27" font="vector" ratio="13" rot="R180"/>
 </element>
-<element name="FD301" library="be_marks" package="CROSSHAIR" value="FIDUCIAL_CROSSHAIR" x="55" y="5" smashed="yes">
+<element name="FD201" library="be_marks" package="CROSSHAIR" value="FIDUCIAL_CROSSHAIR" x="55" y="5" smashed="yes">
 <attribute name="FUNCTION" value="" x="55" y="5" size="1.778" layer="27" display="off"/>
 <attribute name="PART_CODE_EXT" value="" x="55" y="5" size="1.778" layer="27" display="off"/>
@@
 <attribute name="NAME" x="56.5" y="1" size="0.7" layer="26" font="vector" ratio="13" rot="MR0"/>
 </element>
-<element name="FD302" library="be_marks" package="CROSSHAIR" value="FIDUCIAL_CROSSHAIR" x="15" y="45" smashed="yes">
+<element name="FD202" library="be_marks" package="CROSSHAIR" value="FIDUCIAL_CROSSHAIR" x="15" y="45" smashed="yes">
 <attribute name="FUNCTION" value="" x="15" y="45" size="1.778" layer="27" display="off"/>
 <attribute name="PART_CODE_EXT" value="" x="15" y="45" size="1.778" layer="27" display="off"/>
@@
 <attribute name="UPDATED" value="" x="15" y="45" size="1.778" layer="27" display="off"/>
 </element>
-<element name="H303" library="be_holes" package="3.2_PAD" value="HOLE_3.2_PAD" x="5" y="5" smashed="yes">
+<element name="H203" library="be_holes" package="3.2_PAD" value="HOLE_3.2_PAD" x="5" y="5" smashed="yes">
 <attribute name="FUNCTION" value="" x="5" y="5" size="1.778" layer="27" display="off"/>
 <attribute name="PART_CODE_EXT" value="" x="5" y="5" size="1.778" layer="27" display="off"/>
@@
 <attribute name="UPDATED" value="" x="5" y="5" size="1.778" layer="27" display="off"/>
 </element>
-<element name="H304" library="be_holes" package="3.2_PAD" value="HOLE_3.2_PAD" x="5" y="45" smashed="yes">
+<element name="H204" library="be_holes" package="3.2_PAD" value="HOLE_3.2_PAD" x="5" y="45" smashed="yes">
 <attribute name="FUNCTION" value="" x="5" y="45" size="1.778" layer="27" display="off"/>
 <attribute name="PART_CODE_EXT" value="" x="5" y="45" size="1.778" layer="27" display="off"/>
@@
 <attribute name="VALUE" x="34.365" y="29.731" size="1" layer="27" font="vector" ratio="13" rot="R270"/>
 </element>
-<element name="X301" library="be_con_jump" package="T_POWER_JACK_SPC4077" value="" x="9.98" y="35.35" smashed="yes">
+<element name="X201" library="be_con_jump" package="T_POWER_JACK_SPC4077" value="" x="9.98" y="35.35" smashed="yes">
 <attribute name="FUNCTION" value="PWR IN" x="2.2" y="29" size="1" layer="21" font="vector" ratio="15"/>
 <attribute name="PART_CODE_EXT" value="" x="9.98" y="35.35" size="1.778" layer="27" display="off"/>
@@
 <attribute name="VALUE" x="-0.52" y="40.35" size="1" layer="27" font="vector" ratio="13"/>
 </element>
-<element name="H301" library="be_holes" package="3.2_PAD" value="HOLE_3.2_PAD" x="65" y="45" smashed="yes">
+<element name="H201" library="be_holes" package="3.2_PAD" value="HOLE_3.2_PAD" x="65" y="45" smashed="yes">
 <attribute name="FUNCTION" value="" x="65" y="45" size="1" layer="27" font="vector" ratio="13" display="off"/>
 <attribute name="PART_CODE_EXT" value="" x="65" y="45" size="1" layer="27" font="vector" ratio="13" display="off"/>
@@
 <attribute name="UPDATED" value="" x="65" y="45" size="1" layer="27" font="vector" ratio="13" display="off"/>
 </element>
-<element name="H302" library="be_holes" package="3.2_PAD" value="HOLE_3.2_PAD" x="65" y="5" smashed="yes">
+<element name="H202" library="be_holes" package="3.2_PAD" value="HOLE_3.2_PAD" x="65" y="5" smashed="yes">
 <attribute name="FUNCTION" value="" x="65" y="5" size="1" layer="27" font="vector" ratio="13" display="off"/>
 <attribute name="PART_CODE_EXT" value="" x="65" y="5" size="1" layer="27" font="vector" ratio="13" display="off"/>
@@
 <attribute name="UPDATED" value="" x="65" y="5" size="1" layer="27" font="vector" ratio="13" display="off"/>
 </element>
-<element name="C301" library="be_rcl" package="S_6032" value="10u" x="17.4" y="33.8" rot="R270">
+<element name="C201" library="be_rcl" package="S_6032" value="10u" x="17.4" y="33.8" rot="R270">
 <attribute name="FUNCTION" value="" x="17.4" y="33.8" size="1" layer="27" font="vector" ratio="15" rot="R270" display="off"/>
 <attribute name="PART_CODE_EXT" value="" x="17.4" y="33.8" size="1" layer="27" font="vector" ratio="15" rot="R270" display="off"/>
@@
 </element>
 <element name="U$9" library="be_frame" package="A4_LANDSCAPE" value="" x="-158.4" y="-57"/>
-<element name="X302" library="be_con_jump" package="T_MALE_2X10_VERTICAL_GRID_2.54MM" value="MALE_2X10-T-VERTICAL_2.54MM" x="63" y="25" smashed="yes" rot="R270">
+<element name="X202" library="be_con_jump" package="T_MALE_2X10_VERTICAL_GRID_2.54MM" value="MALE_2X10-T-VERTICAL_2.54MM" x="63" y="25" smashed="yes" rot="R270">
 <attribute name="FUNCTION" value="TO SHIELD" x="59.8" y="13" size="1.5" layer="21" font="vector" ratio="15" rot="R90"/>
 <attribute name="PART_CODE_EXT" value="" x="63" y="25" size="1.5" layer="27" font="vector" ratio="15" rot="R270" display="off"/>
@@
 <contactref element="C101" pad="1"/>
 <contactref element="IC101" pad="14"/>
-<contactref element="X301" pad="3"/>
+<contactref element="X201" pad="3"/>
 <wire x1="37.95" y1="34" x2="38.55" y2="34.6" width="0.15" layer="1"/>
 <wire x1="38.55" y1="34.6" x2="39.2" y2="34.6" width="0.15" layer="1"/>
@@
 <via x="39.2" y="33.4" extent="1-16" drill="0.3"/>
 <via x="39.2" y="34.6" extent="1-16" drill="0.3"/>
-<contactref element="C301" pad="+"/>
+<contactref element="C201" pad="+"/>
 <wire x1="17.4" y1="36.3" x2="16.45" y2="35.35" width="1" layer="1"/>
 <wire x1="16.45" y1="35.35" x2="12.98" y2="35.35" width="1" layer="1"/>
@@
 <contactref element="C101" pad="2"/>
 <contactref element="IC101" pad="7"/>
-<contactref element="X301" pad="1"/>
+<contactref element="X201" pad="1"/>
 <polygon width="0.15" layer="16">
 <vertex x="0" y="50"/>
@@
 <via x="34.8" y="33.4" extent="1-16" drill="0.3"/>
 <via x="34.8" y="34.6" extent="1-16" drill="0.3"/>
-<contactref element="C301" pad="-"/>
+<contactref element="C201" pad="-"/>
 <wire x1="17.4" y1="31.3" x2="18.3" y2="32.2" width="0.15" layer="1"/>
 <wire x1="18.3" y1="32.2" x2="19.2" y2="32.2" width="0.15" layer="1"/>
@@
 <via x="19.2" y="30.4" extent="1-16" drill="0.3"/>
 <via x="19.2" y="32.2" extent="1-16" drill="0.3"/>
-<contactref element="X302" pad="1"/>
-<contactref element="X302" pad="3"/>
+<contactref element="X202" pad="1"/>
+<contactref element="X202" pad="3"/>
 </signal>
 <signal name="MCU_CLK">
@@
 <wire x1="44.4" y1="21.6" x2="44.8" y2="22" width="0.15" layer="1"/>
 <wire x1="44.8" y1="22" x2="44.8" y2="27" width="0.15" layer="1"/>
-<contactref element="X302" pad="2"/>
+<contactref element="X202" pad="2"/>
 <wire x1="44.8" y1="27" x2="53" y2="35.2" width="0.15" layer="1"/>
 <wire x1="53" y1="35.2" x2="63.2" y2="35.2" width="0.15" layer="1"/>
@@
 <wire x1="44.66" y1="20.46" x2="45.6" y2="21.4" width="0.3" layer="1"/>
 <wire x1="45.6" y1="21.4" x2="45.6" y2="25.2" width="0.3" layer="1"/>
-<contactref element="X302" pad="4"/>
+<contactref element="X202" pad="4"/>
 <wire x1="45.6" y1="25.2" x2="53" y2="32.6" width="0.3" layer="1"/>
 <wire x1="53" y1="32.6" x2="63" y2="32.6" width="0.3" layer="1"/>
