File: eagle/demo/shield.brd (EAGLE design)
At the start: 70 x 50 mm, 16 parts, among them X1 MALE_2X1-T-VERTICAL, X301 MALE_2X1-T-VERTICAL, X302 MALE_2X10-T-VERTICAL_2.54MM

Commit message: kbd module
Connections:
- net CORE_CLK renamed MCU_CLK
- net CORE_QD renamed MCU_QD
Changed lines of the file:
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@@
 <via x="7.8" y="29" extent="1-16" drill="0.3"/>
 </signal>
-<signal name="CORE_CLK">
+<signal name="MCU_CLK">
 <contactref element="X302" pad="2"/>
 <contactref element="N2" pad="2"/>
@@
 <wire x1="62.84" y1="35" x2="56.3" y2="35" width="0.15" layer="1"/>
 </signal>
-<signal name="CORE_QD">
+<signal name="MCU_QD">
 <contactref element="X302" pad="4"/>
 <contactref element="N1" pad="2"/>

Commit message: fixed prefixes
Connections:
- net BACKEND_DRV_IN renamed LED_DRV_IN
- net BACKEND_KBD_OUT renamed KBD_OUT
Changed lines of the file:
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@@
 <wire x1="63.18" y1="32.8" x2="56.3" y2="32.8" width="0.3" layer="1"/>
 </signal>
-<signal name="BACKEND_DRV_IN">
+<signal name="LED_DRV_IN">
 <contactref element="X301" pad="2"/>
 <contactref element="N1" pad="1"/>
@@
 <wire x1="52.8" y1="29.8" x2="52.8" y2="32.8" width="0.15" layer="1"/>
 </signal>
-<signal name="BACKEND_KBD_OUT">
+<signal name="KBD_OUT">
 <contactref element="N2" pad="1"/>
 <contactref element="X1" pad="2"/>

Commit message: fix partcodes
Parts:
- LED301: value (none) -> green
- LED401: value (none) -> red
- renumbered FD1 to FD101, FD2 to FD102, H1 to H103, H2 to H104, H3 to H101, H4 to H102, LED3 to LED401, LED4 to LED301, N1 to N201, N2 to N202, R3 to R401, R4 to R301, X1 to X401, X302 to X101
