File: eagle/demo/shield_2x_driver.brd (EAGLE design)
At the start: 70 x 50 mm, 20 parts, among them X1 MALE_2X1-T-VERTICAL, X2 MALE_2X1-T-VERTICAL, X301 MALE_2X1-T-VERTICAL, X302 MALE_2X10-T-VERTICAL_2.54MM

Commit message: fix partcodes
Parts:
- LED301, LED401: value (none) -> green
- LED501: value (none) -> red
- renumbered FD1 to FD101, FD2 to FD102, H1 to H103, H2 to H104, H3 to H101, H4 to H102, LED1 to LED401, LED3 to LED501, LED4 to LED301, N1 to N202, N2 to N203, N3 to N201, R1 to R401, R3 to R501, R4 to R301, X1 to X501, X2 to X401, X302 to X101

Commit message: fix net names
Connections:
- net LED_DRV_IN_1 renamed LED_DRV_1_IN
- net LED_DRV_IN_2 renamed LED_DRV_2_IN
- net SH_DBG_DRV_1 renamed SH_DBG_1_DRV
- net SH_DBG_DRV_2 renamed SH_DBG_2_DRV
Changed lines of the file:
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@@
 <wire x1="15.05" y1="34" x2="11.05" y2="34" width="0.15" layer="1"/>
 </signal>
-<signal name="SH_DBG_DRV_1">
+<signal name="SH_DBG_1_DRV">
 <contactref element="R301" pad="1"/>
 <contactref element="LED301" pad="A"/>
 <wire x1="15.05" y1="29" x2="11.05" y2="29" width="0.15" layer="1"/>
 </signal>
-<signal name="LED_DRV_IN_2">
+<signal name="LED_DRV_2_IN">
 <contactref element="R401" pad="2"/>
 <contactref element="X401" pad="2"/>
@@
 <wire x1="57.4" y1="45" x2="57.27" y2="45" width="0.15" layer="1"/>
 </signal>
-<signal name="SH_DBG_DRV_2">
+<signal name="SH_DBG_2_DRV">
 <contactref element="R401" pad="1"/>
 <contactref element="LED401" pad="A"/>
 <wire x1="15.05" y1="24" x2="11.05" y2="24" width="0.15" layer="1"/>
 </signal>
-<signal name="LED_DRV_IN_1">
+<signal name="LED_DRV_1_IN">
 <contactref element="X301" pad="2"/>
 <contactref element="R301" pad="2"/>
