File: eagle_demo/demo/keyboard.sch (EAGLE design)
At the start: 8 parts, among them X1 CLAMP_1X2-T-2.5MM, X2 CLAMP_1X2-T-2.5MM

Commit message: step 1.4 keyboard layout
Parts:
- S1: FUNCTION (none) -> ACTIVATE LIGHT
- X2: FUNCTION (none) -> SHIELD CTRL IN
Changed lines of the file:
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@@
 <attribute name="FUNCTION" value="PWR IN"/>
 </part>
-<part name="S1" library="be_switch" deviceset="PUSH_BUTTON" device="_S_6X6MM"/>
+<part name="S1" library="be_switch" deviceset="PUSH_BUTTON" device="_S_6X6MM">
+<attribute name="FUNCTION" value="ACTIVATE LIGHT"/>
+</part>
 <part name="GND1" library="be_supply" deviceset="GND" device=""/>
 <part name="R1" library="be_rcl" deviceset="R" device="_S_0805"/>
 <part name="FRAME_DEVELOPMENT2" library="be_frame" deviceset="A4_LANDSCAPE_DEVELOPMENT" device=""/>
-<part name="X2" library="be_con_jump" deviceset="CLAMP_1X2" device="-T-2.5MM"/>
+<part name="X2" library="be_con_jump" deviceset="CLAMP_1X2" device="-T-2.5MM">
+<attribute name="FUNCTION" value="SHIELD CTRL IN"/>
+</part>
 <part name="GND2" library="be_supply" deviceset="GND" device=""/>
 </parts>
