File: eagle_demo/demo/shield.sch (EAGLE design)
At the start: 12 parts, among them X301 MALE_2X1-T-VERTICAL, X302 MALE_2X10-T-VERTICAL_2.54MM

Commit message: step 1.3 shield schematic updated
Parts:
- added LED1: (no value), be_opt:LED_S_0805
- added R1: 330, be_rcl:R_S_0805
- added X2: CLAMP_1X2-T-2.5MM, be_con_jump:CLAMP_1X2-T-2.5MM
Connections:
- new net KBD_OUT: N2.1, R1.2, X2.2
- new net SH_KBD_DBG: LED1.A, R1.1
- net GND: now also LED1.C, X2.1
Changed lines of the file:
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@@
 <part name="LED4" library="be_opt" deviceset="LED" device="_S_0805"/>
 <part name="GND6" library="be_supply" deviceset="GND" device=""/>
+<part name="FRAME_DEVELOPMENT3" library="be_frame" deviceset="A4_LANDSCAPE_DEVELOPMENT" device=""/>
+<part name="X2" library="be_con_jump" deviceset="CLAMP_1X2" device="-T-2.5MM"/>
+<part name="GND2" library="be_supply" deviceset="GND" device=""/>
+<part name="R1" library="be_rcl" deviceset="R" device="_S_0805" value="330"/>
+<part name="LED1" library="be_opt" deviceset="LED" device="_S_0805">
+<attribute name="FUNCTION" value="KBD BUTTON PRESSED"/>
+</part>
+<part name="GND3" library="be_supply" deviceset="GND" device=""/>
 </parts>
 <sheets>
@@
 </segment>
 </net>
+<net name="KBD_OUT" class="0">
+<segment>
+<pinref part="N2" gate="G$1" pin="1"/>
+<wire x1="172.72" y1="45.72" x2="180.34" y2="45.72" width="0.1524" layer="91"/>
+<label x="180.34" y="45.72" size="1.27" layer="95" font="fixed" xref="yes"/>
+</segment>
+</net>
 </nets>
 </sheet>
@@
 </segment>
 </net>
+</nets>
+</sheet>
+<sheet>
+<description>connector KBD module</description>
+<plain>
+</plain>
+<instances>
+<instance part="FRAME_DEVELOPMENT3" gate="G$1" x="0" y="0"/>
+<instance part="X2" gate="G$1" x="38.1" y="121.92" rot="R180"/>
+<instance part="GND2" gate="1" x="50.8" y="114.3"/>
+<instance part="R1" gate="G$1" x="55.88" y="83.82" rot="R90"/>
+<instance part="LED1" gate="G$1" x="55.88" y="73.66">
+<attribute name="FUNCTION" x="58.42" y="71.12" size="1.27" layer="96" font="fixed"/>
+</instance>
+<instance part="GND3" gate="1" x="55.88" y="63.5"/>
+</instances>
+<busses>
+</busses>
+<nets>
+<net name="GND" class="0">
+<segment>
+<pinref part="X2" gate="G$1" pin="1"/>
+<pinref part="GND2" gate="1" pin="GND"/>
+<wire x1="40.64" y1="119.38" x2="50.8" y2="119.38" width="0.1524" layer="91"/>
+<wire x1="50.8" y1="119.38" x2="50.8" y2="116.84" width="0.1524" layer="91"/>
+</segment>
+<segment>
+<pinref part="LED1" gate="G$1" pin="C"/>
+<pinref part="GND3" gate="1" pin="GND"/>
+<wire x1="55.88" y1="66.04" x2="55.88" y2="68.58" width="0.1524" layer="91"/>
+</segment>
+</net>
+<net name="KBD_OUT" class="0">
+<segment>
+<pinref part="X2" gate="G$1" pin="2"/>
+<wire x1="40.64" y1="121.92" x2="60.96" y2="121.92" width="0.1524" layer="91"/>
+<label x="60.96" y="121.92" size="1.27" layer="95" font="fixed" xref="yes"/>
+</segment>
+<segment>
+<pinref part="R1" gate="G$1" pin="2"/>
+<wire x1="55.88" y1="88.9" x2="55.88" y2="91.44" width="0.1524" layer="91"/>
+<wire x1="55.88" y1="91.44" x2="35.56" y2="91.44" width="0.1524" layer="91"/>
+<label x="36.195" y="92.075" size="1.27" layer="95" font="fixed"/>
+</segment>
+</net>
+<net name="SH_KBD_DBG" class="0">
+<segment>
+<pinref part="R1" gate="G$1" pin="1"/>
+<pinref part="LED1" gate="G$1" pin="A"/>
+<wire x1="55.88" y1="78.74" x2="55.88" y2="76.2" width="0.1524" layer="91"/>
+<label x="55.88" y="77.47" size="1.27" layer="95" font="fixed" xref="yes"/>
+</segment>
+</net>

Commit message: step 1.5 shield layout
Parts:
- LED4: FUNCTION (none) -> LIGHT ACTIVE
Changed lines of the file:
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@@
 <part name="H4" library="be_holes" deviceset="HOLE" device="_3.2_PAD"/>
 <part name="R4" library="be_rcl" deviceset="R" device="_S_0805" value="330"/>
-<part name="LED4" library="be_opt" deviceset="LED" device="_S_0805"/>
+<part name="LED4" library="be_opt" deviceset="LED" device="_S_0805">
+<attribute name="FUNCTION" value="LIGHT ACTIVE"/>
+</part>
 <part name="GND6" library="be_supply" deviceset="GND" device=""/>
 <part name="FRAME_DEVELOPMENT3" library="be_frame" deviceset="A4_LANDSCAPE_DEVELOPMENT" device=""/>
