File: eagle_demo/demo/product.sch (EAGLE design)
At the start: 45 parts, among them IC101 MCU, T101 BC548C, X1 MALE_2X10-T-VERTICAL_2.54MM, X2 MALE_2X1-T-VERTICAL, X3 CLAMP_1X2-T-2.5MM, X302 MALE_2X10-T-VERTICAL_2.54MM, X4 CLAMP_1X2-T-2.5MM, X5 MALE_2X1-T-VERTICAL, X6 CLAMP_1X2-T-2.5MM, X7 CLAMP_1X2-T-2.5MM, X8 CLAMP_1X2-T-2.5MM

Commit message: step 2.1.2 dev pages removed
Parts:
- removed C301: 10U, be_rcl:C_POL_S_6032
- removed FD1, FD2, FD3, FD301, FD302, FD4, FD5, FD6: FIDUCIAL_CROSSHAIR, be_marks:FIDUCIAL_CROSSHAIR
- removed H1, H2, H3, H301, H302, H303, H304, H4, H5, H6, H7, H8: HOLE_3.2_PAD, be_holes:HOLE_3.2_PAD
- removed LED1, LED4: (no value), be_opt:LED_S_0805
- removed R1, R4: 330, be_rcl:R_S_0805
- removed X1, X302: MALE_2X10-T-VERTICAL_2.54MM, be_con_jump:MALE_2X10-T-VERTICAL_2.54MM
- removed X2, X5: MALE_2X1-T-VERTICAL, be_con_jump:MALE_2X1-T-VERTICAL
- removed X3, X6, X7, X8: CLAMP_1X2-T-2.5MM, be_con_jump:CLAMP_1X2-T-2.5MM
- removed X301: (no value), be_con_jump:POWER_JACK-T-0
Connections:
- removed net SH_DBG_DRV: LED4.A, R4.1
- removed net SH_KBD_DBG: LED1.A, R1.1
- net GND: no longer C301.-, LED1.C, LED4.C, X1.1, X1.3, X2.1, X3.1, X301.1, X302.1, X302.3, X5.1, X6.1, X7.1, X8.1
- net KBD_OUT: no longer R1.2, X3.2, X8.2
- net LED_DRV_IN: no longer R4.2, X2.2, X5.2
- net MCU_CLK: no longer X1.2, X302.2
- net MCU_QD: no longer X1.4, X302.4
- net P5V: no longer C301.+, X301.3, X6.2, X7.2

Commit message: step 2.2 reduce routing
Parts:
- removed N1: NET_CHANGER-S-0.3MM, be_con_jump:NET_CHANGER-S-0.3MM
- removed N2: NET_CHANGER-S-0.15MM, be_con_jump:NET_CHANGER-S-0.15MM
Connections:
- removed net MCU_CLK: IC101G$1.C1, N2.2
- removed net MCU_QD: IC101G$1.QD, N1.2
- net KBD_OUT: now also IC101G$1.C1; no longer N2.1
- net LED_DRV_IN: now also IC101G$1.QD; no longer N1.1
Changed lines of the file:
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@@
 <part name="U$3" library="be_info" deviceset="ARROW_1" device=""/>
 <part name="U$4" library="be_info" deviceset="ARROW_1" device=""/>
-<part name="FRAME_NET_CHANGERS1" library="be_frame" deviceset="A4_LANDSCAPE_NET_CHANGERS" device=""/>
-<part name="N1" library="be_con_jump" deviceset="NET_CHANGER" device="-S-0.3MM"/>
-<part name="U$6" library="be_info" deviceset="ARROW_1" device=""/>
-<part name="U$7" library="be_info" deviceset="ARROW_1" device=""/>
-<part name="N2" library="be_con_jump" deviceset="NET_CHANGER" device="-S-0.15MM" value="NET_CHANGER-S-0.15MM"/>
-<part name="U$8" library="be_info" deviceset="ARROW_1" device=""/>
 <part name="FRAME_PRODUCT2" library="be_frame" deviceset="A4_LANDSCAPE_PRODUCT" device="">
 <attribute name="DESCRIPTION" value="LED driver"/>
@@
 </segment>
 </net>
-<net name="MCU_CLK" class="0">
+<net name="KBD_OUT" class="0">
 <segment>
 <pinref part="IC101" gate="G$1" pin="C1"/>
@@
 </segment>
 </net>
-<net name="MCU_QD" class="0">
+<net name="LED_DRV_IN" class="0">
 <segment>
 <pinref part="IC101" gate="G$1" pin="QD"/>
@@
 </segment>
 </net>
-</nets>
-</sheet>
-<sheet>
-<description>routing</description>
-<plain>
-</plain>
-<instances>
-<instance part="FRAME_NET_CHANGERS1" gate="G$1" x="0" y="0"/>
-<instance part="N1" gate="G$1" x="165.1" y="53.34" rot="MR0"/>
-<instance part="U$6" gate="G$1" x="175.26" y="53.34" rot="R180"/>
-<instance part="U$7" gate="G$1" x="152.4" y="53.34" rot="R180"/>
-<instance part="N2" gate="G$1" x="165.1" y="45.72" rot="MR0"/>
-<instance part="U$8" gate="G$1" x="154.94" y="45.72"/>
-</instances>
-<busses>
-</busses>
-<nets>
-<net name="MCU_QD" class="0">
-<segment>
-<pinref part="N1" gate="G$1" pin="2"/>
-<wire x1="157.48" y1="53.34" x2="149.86" y2="53.34" width="0.1524" layer="91"/>
-<label x="149.86" y="53.34" size="1.27" layer="95" font="fixed" rot="R180" xref="yes"/>
-</segment>
-</net>
-<net name="LED_DRV_IN" class="0">
-<segment>
-<pinref part="N1" gate="G$1" pin="1"/>
-<wire x1="172.72" y1="53.34" x2="180.34" y2="53.34" width="0.1524" layer="91"/>
-<label x="180.34" y="53.34" size="1.27" layer="95" font="fixed" xref="yes"/>
-</segment>
-</net>
-<net name="MCU_CLK" class="0">
-<segment>
-<pinref part="N2" gate="G$1" pin="2"/>
-<wire x1="157.48" y1="45.72" x2="149.86" y2="45.72" width="0.1524" layer="91"/>
-<label x="149.86" y="45.72" size="1.27" layer="95" font="fixed" rot="R180" xref="yes"/>
-</segment>
-</net>
-<net name="KBD_OUT" class="0">
-<segment>
-<pinref part="N2" gate="G$1" pin="1"/>
-<wire x1="172.72" y1="45.72" x2="180.34" y2="45.72" width="0.1524" layer="91"/>
-<label x="180.34" y="45.72" size="1.27" layer="95" font="fixed" xref="yes"/>
-</segment>
-</net>

Commit message: step 2.3 product layout placement
Parts:
- C1: device be_rcl:C_POL_S_6032 -> be_rcl:C_POL_S_3216-18
- C101: device be_rcl:C_S_0805 -> be_rcl:C_S_0603
- IC101: device be_logic:7495A -> be_logic:7495D
- R101, R102, R2: device be_rcl:R_S_0805 -> be_rcl:R_S_0603
Changed lines of the file:
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@@
 <grid distance="0.1" unitdist="inch" unit="inch" style="lines" multiple="1" display="no" altdistance="0.025" altunitdist="inch" altunit="inch"/>
 <layers>
-<layer number="1" name="Top" color="4" fill="1" visible="no" active="no"/>
-<layer number="2" name="Route2" color="1" fill="3" visible="no" active="no"/>
-<layer number="3" name="Route3" color="4" fill="3" visible="no" active="no"/>
-<layer number="4" name="Route4" color="1" fill="4" visible="no" active="no"/>
-<layer number="5" name="Route5" color="4" fill="4" visible="no" active="no"/>
-<layer number="6" name="Route6" color="1" fill="8" visible="no" active="no"/>
-<layer number="7" name="Route7" color="4" fill="8" visible="no" active="no"/>
-<layer number="8" name="Route8" color="1" fill="2" visible="no" active="no"/>
-<layer number="9" name="Route9" color="4" fill="2" visible="no" active="no"/>
-<layer number="10" name="Route10" color="1" fill="7" visible="no" active="no"/>
-<layer number="11" name="Route11" color="4" fill="7" visible="no" active="no"/>
-<layer number="12" name="Route12" color="1" fill="5" visible="no" active="no"/>
-<layer number="13" name="Route13" color="4" fill="5" visible="no" active="no"/>
-<layer number="14" name="Route14" color="1" fill="6" visible="no" active="no"/>
-<layer number="15" name="Route15" color="4" fill="6" visible="no" active="no"/>
-<layer number="16" name="Bottom" color="1" fill="1" visible="no" active="no"/>
-<layer number="17" name="Pads" color="2" fill="1" visible="no" active="no"/>
-<layer number="18" name="Vias" color="2" fill="1" visible="no" active="no"/>
-<layer number="19" name="Unrouted" color="6" fill="1" visible="no" active="no"/>
-<layer number="20" name="Dimension" color="15" fill="1" visible="no" active="no"/>
-<layer number="21" name="tPlace" color="7" fill="1" visible="no" active="no"/>
-<layer number="22" name="bPlace" color="7" fill="1" visible="no" active="no"/>
-<layer number="23" name="tOrigins" color="15" fill="1" visible="no" active="no"/>
-<layer number="24" name="bOrigins" color="15" fill="1" visible="no" active="no"/>
-<layer number="25" name="tNames" color="7" fill="1" visible="no" active="no"/>
-<layer number="26" name="bNames" color="7" fill="1" visible="no" active="no"/>
-<layer number="27" name="tValues" color="7" fill="1" visible="no" active="no"/>
-<layer number="28" name="bValues" color="7" fill="1" visible="no" active="no"/>
+<layer number="1" name="Top" color="4" fill="1" visible="yes" active="no"/>
+<layer number="2" name="Route2" color="1" fill="3" visible="yes" active="no"/>
+<layer number="3" name="Route3" color="4" fill="3" visible="yes" active="no"/>
+<layer number="4" name="Route4" color="1" fill="4" visible="yes" active="no"/>
+<layer number="5" name="Route5" color="4" fill="4" visible="yes" active="no"/>
+<layer number="6" name="Route6" color="1" fill="8" visible="yes" active="no"/>
+<layer number="7" name="Route7" color="4" fill="8" visible="yes" active="no"/>
+<layer number="8" name="Route8" color="1" fill="2" visible="yes" active="no"/>
+<layer number="9" name="Route9" color="4" fill="2" visible="yes" active="no"/>
+<layer number="10" name="Route10" color="1" fill="7" visible="yes" active="no"/>
+<layer number="11" name="Route11" color="4" fill="7" visible="yes" active="no"/>
+<layer number="12" name="Route12" color="1" fill="5" visible="yes" active="no"/>
+<layer number="13" name="Route13" color="4" fill="5" visible="yes" active="no"/>
+<layer number="14" name="Route14" color="1" fill="6" visible="yes" active="no"/>
+<layer number="15" name="Route15" color="4" fill="6" visible="yes" active="no"/>
+<layer number="16" name="Bottom" color="1" fill="1" visible="yes" active="no"/>
+<layer number="17" name="Pads" color="2" fill="1" visible="yes" active="no"/>
+<layer number="18" name="Vias" color="2" fill="1" visible="yes" active="no"/>
+<layer number="19" name="Unrouted" color="6" fill="1" visible="yes" active="no"/>
+<layer number="20" name="Dimension" color="15" fill="1" visible="yes" active="no"/>
+<layer number="21" name="tPlace" color="7" fill="1" visible="yes" active="no"/>
+<layer number="22" name="bPlace" color="7" fill="1" visible="yes" active="no"/>
+<layer number="23" name="tOrigins" color="15" fill="1" visible="yes" active="no"/>
+<layer number="24" name="bOrigins" color="15" fill="1" visible="yes" active="no"/>
+<layer number="25" name="tNames" color="7" fill="1" visible="yes" active="no"/>
+<layer number="26" name="bNames" color="7" fill="1" visible="yes" active="no"/>
+<layer number="27" name="tValues" color="7" fill="1" visible="yes" active="no"/>
+<layer number="28" name="bValues" color="7" fill="1" visible="yes" active="no"/>
 <layer number="29" name="tStop" color="7" fill="3" visible="no" active="no"/>
 <layer number="30" name="bStop" color="7" fill="6" visible="no" active="no"/>
@@
 <layer number="35" name="tGlue" color="7" fill="4" visible="no" active="no"/>
 <layer number="36" name="bGlue" color="7" fill="5" visible="no" active="no"/>
-<layer number="37" name="tTest" color="7" fill="1" visible="no" active="no"/>
-<layer number="38" name="bTest" color="7" fill="1" visible="no" active="no"/>
+<layer number="37" name="tTest" color="7" fill="1" visible="yes" active="no"/>
+<layer number="38" name="bTest" color="7" fill="1" visible="yes" active="no"/>
 <layer number="39" name="tKeepout" color="4" fill="11" visible="no" active="no"/>
 <layer number="40" name="bKeepout" color="1" fill="11" visible="no" active="no"/>
@@
 <layer number="44" name="Drills" color="7" fill="1" visible="no" active="no"/>
 <layer number="45" name="Holes" color="7" fill="1" visible="no" active="no"/>
-<layer number="46" name="Milling" color="3" fill="1" visible="no" active="no"/>
-<layer number="47" name="Measures" color="7" fill="1" visible="no" active="no"/>
-<layer number="48" name="Document" color="7" fill="1" visible="no" active="no"/>
-<layer number="49" name="Reference" color="7" fill="1" visible="no" active="no"/>
-<layer number="50" name="dxf" color="7" fill="1" visible="no" active="no"/>
-<layer number="51" name="tDocu" color="7" fill="1" visible="no" active="no"/>
-<layer number="52" name="bDocu" color="7" fill="1" visible="no" active="no"/>
-<layer number="53" name="tGND_GNDA" color="7" fill="1" visible="no" active="no"/>
-<layer number="54" name="bGND_GNDA" color="7" fill="1" visible="no" active="no"/>
-<layer number="56" name="wert" color="7" fill="1" visible="no" active="no"/>
-<layer number="57" name="HEIGHT" color="7" fill="1" visible="no" active="no"/>
-<layer number="58" name="DEPTH" color="7" fill="1" visible="no" active="no"/>
+<layer number="46" name="Milling" color="3" fill="1" visible="yes" active="no"/>
+<layer number="47" name="Measures" color="7" fill="1" visible="yes" active="no"/>
+<layer number="48" name="Document" color="7" fill="1" visible="yes" active="no"/>
+<layer number="49" name="Reference" color="7" fill="1" visible="yes" active="no"/>
+<layer number="50" name="dxf" color="7" fill="1" visible="yes" active="no"/>
+<layer number="51" name="tDocu" color="7" fill="1" visible="yes" active="no"/>
+<layer number="52" name="bDocu" color="7" fill="1" visible="yes" active="no"/>
+<layer number="53" name="tGND_GNDA" color="7" fill="1" visible="yes" active="no"/>
+<layer number="54" name="bGND_GNDA" color="7" fill="1" visible="yes" active="no"/>
+<layer number="56" name="wert" color="7" fill="1" visible="yes" active="no"/>
+<layer number="57" name="HEIGHT" color="7" fill="1" visible="yes" active="no"/>
+<layer number="58" name="DEPTH" color="7" fill="1" visible="yes" active="no"/>
 <layer number="90" name="Modules" color="5" fill="1" visible="yes" active="yes"/>
 <layer number="91" name="Nets" color="2" fill="1" visible="yes" active="yes"/>
@@
 <attribute name="DESCRIPTION" value="core / MCU"/>
 </part>
-<part name="IC101" library="be_logic" deviceset="74*95" device="A" value="MCU"/>
-<part name="C101" library="be_rcl" deviceset="C" device="_S_0805" value="100n"/>
+<part name="IC101" library="be_logic" deviceset="7495" device="D" value="MCU"/>
+<part name="C101" library="be_rcl" deviceset="C" device="_S_0603" value="100n"/>
 <part name="GND1" library="be_supply" deviceset="GND" device=""/>
 <part name="GND2" library="be_supply" deviceset="GND" device=""/>
@@
 <attribute name="DESCRIPTION" value="LED driver"/>
 </part>
-<part name="R101" library="be_rcl" deviceset="R" device="_S_0805" value="2k2"/>
+<part name="R101" library="be_rcl" deviceset="R" device="_S_0603" value="2k2"/>
 <part name="T101" library="be_transistor" deviceset="NPN" device="_S_SOT23" value="BC548C"/>
-<part name="R102" library="be_rcl" deviceset="R" device="_S_0805" value="100"/>
+<part name="R102" library="be_rcl" deviceset="R" device="_S_0603" value="100"/>
 <part name="GND11" library="be_supply" deviceset="GND" device=""/>
-<part name="C1" library="be_rcl" deviceset="C_POL" device="_S_6032" value="100n"/>
+<part name="C1" library="be_rcl" deviceset="C_POL" device="_S_3216-18" value="100n"/>
 <part name="GND12" library="be_supply" deviceset="GND" device=""/>
 <part name="X4" library="be_con_jump" deviceset="CLAMP_1X2" device="-T-2.5MM">
@@
 </part>
 <part name="GND16" library="be_supply" deviceset="GND" device=""/>
-<part name="R2" library="be_rcl" deviceset="R" device="_S_0805"/>
+<part name="R2" library="be_rcl" deviceset="R" device="_S_0603"/>
 </parts>
 <sheets>
