File: eagle_demo/demo/template.sch (EAGLE design)
At the start: 5 parts, among them X1 CLAMP_1X2-T-2.5MM

Commit message: fix template
Changed lines of the file:
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@@
 </classes>
 <parts>
-<part name="FRAME_PRODUCT1" library="be_frame" deviceset="A4_LANDSCAPE_PRODUCT" device="">
-<attribute name="DESCRIPTION" value="LED driver"/>
-</part>
+<part name="FRAME_PRODUCT1" library="be_frame" deviceset="A4_LANDSCAPE_PRODUCT" device=""/>
 <part name="FRAME_DEVELOPMENT1" library="be_frame" deviceset="A4_LANDSCAPE_DEVELOPMENT" device=""/>
-<part name="FRAME_NET_CHANGERS1" library="be_frame" deviceset="A4_LANDSCAPE_NET_CHANGERS" device=""/>
 <part name="FD301" library="be_marks" deviceset="FIDUCIAL" device="_CROSSHAIR"/>
 <part name="FD302" library="be_marks" deviceset="FIDUCIAL" device="_CROSSHAIR"/>
@@
 </instances>
 <busses>
-</busses>
-<nets>
-</nets>
-</sheet>
-<sheet>
-<plain>
-</plain>
-<instances>
-<instance part="FRAME_NET_CHANGERS1" gate="G$1" x="0" y="0"/>
-</instances>
-<busses>
